File: kb.kicad_pcb (KiCad board)
At the start: 2 copper layers, 297.6 x 78.5 mm, 120 parts, among them J1 OLED, SW1 SW_PUSH, SW10 SW_PUSH, SW11 SW_PUSH, SW12 SW_PUSH, SW13 SW_PUSH, SW14 SW_PUSH, SW15 SW_PUSH, SW16 SW_PUSH, SW17 SW_PUSH, SW18 SW_PUSH, SW19 SW_PUSH, SW2 SW_PUSH, SW20 SW_PUSH, SW21 SW_PUSH, SW22 SW_PUSH, SW23 SW_PUSH, SW24 SW_PUSH, SW25 SW_PUSH, SW26 SW_PUSH, SW27 SW_PUSH, SW28 SW_PUSH, SW29 SW_PUSH, SW3 SW_PUSH, SW30 SW_PUSH, SW31 SW_PUSH, SW32 SW_PUSH, SW33 SW_PUSH, SW34 SW_PUSH, SW35 SW_PUSH, SW36 SW_PUSH, SW37 SW_PUSH, SW38 SW_PUSH, SW39 SW_PUSH, SW4 SW_PUSH, SW40 SW_PUSH, SW41 SW_PUSH, SW42 SW_PUSH, SW43 SW_PUSH, SW44 SW_PUSH, SW45 SW_PUSH, SW46 SW_PUSH, SW47 SW_PUSH, SW48 SW_PUSH, SW49 SW_Push, SW5 SW_PUSH, SW6 SW_PUSH, SW7 SW_PUSH, SW8 SW_PUSH, SW9 SW_PUSH, U1 ProMicro

Commit message: modify silk
Other:
- board text added: "PCB designed by ... T.komiyama"
- board text added: "Rev. 1.1"
- board text added: "kmykbd - row-staggered 40% keyboard."
- board text removed: "PCB designed by ... TK"
- board text removed: "Rev. 0.1"
- board text removed: "row-staggered 48 keys 4x12-layout keyboard."
Changed lines of the file:
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@@
     (pad 3 thru_hole circle (at 3.5 2.5 90) (size 1.8 1.8) (drill 1.3) (layers *.Cu *.Mask))
   )
-  (gr_text "PCB designed by ... TK" (at 109.22 167.41 -45) (layer F.SilkS)
+  (gr_text "PCB designed by ... T.komiyama" (at 106.76 164.95 -45) (layer F.SilkS)
     (effects (font (size 1 1) (thickness 0.15)) (justify mirror))
   )
@@
   (gr_arc (start 97.609623 155.407463) (end 95.4396 155.407463) (angle -48.79116569) (layer Edge.Cuts) (width 0.05))
   (gr_line (start 96.18 157.04) (end 114.042927 174.898227) (layer Edge.Cuts) (width 0.05))
-  (gr_text "Rev. 0.1" (at 386.9 124.27 90) (layer F.SilkS)
+  (gr_text "Rev. 1.1" (at 386.12 126.37 90) (layer F.SilkS)
     (effects (font (size 1.6 1.6) (thickness 0.3)))
   )
-  (gr_text "row-staggered 48 keys 4x12-layout keyboard." (at 390.22 146.11 90) (layer F.SilkS)
+  (gr_text "kmykbd - row-staggered 40% keyboard." (at 390.22 146.11 90) (layer F.SilkS)
     (effects (font (size 1.6 1.6) (thickness 0.3)))
   )

Commit message: remove front LED pattern
Parts:
- D49, D50, D51, D52, D53, D54, D55, D56, D57, D58, D59, D60, D61, D62: footprint Ergodash_Rev1:WS2812B-5 -> Rev1:WS2812B-5_B_2
- moved SW49 3.18 mm to (101.0, 141.8)
- moved D49 2.58 mm to (106.2, 106.8)
- moved D50 1.86 mm to (107.8, 141.5)
Connections:
- D62 pad 2: Net-(D62-Pad2) -> (no net)
- U1 pad 2: Net-(U1-Pad2) -> (no net)
- U1 pad 24: Net-(U1-Pad24) -> (no net)
Routing:
- net VCC: track 675.3 -> 448.7 mm, vias 4 -> 0
- net GND: track 685.0 -> 464.6 mm, vias 4 -> 0
- net row3: track 242.5 -> 211.6 mm, vias 0 -> 1
- net Net-(D57-Pad2): track 80.0 -> 49.6 mm, vias 1 -> 0
- net Net-(D52-Pad2): track 75.0 -> 46.8 mm, vias 1 -> 0
- net Net-(D61-Pad2): track 68.8 -> 40.7 mm, vias 1 -> 0
- net Net-(D56-Pad2): track 87.1 -> 61.1 mm, vias 1 -> 0
- net Net-(D58-Pad2): track 69.5 -> 44.8 mm, vias 1 -> 0
- net Net-(D53-Pad2): track 62.3 -> 38.8 mm, vias 1 -> 0
- net Net-(D51-Pad2): track 50.6 -> 30.0 mm, vias 1 -> 0
- net Net-(D55-Pad2): track 58.1 -> 37.5 mm, vias 1 -> 0
- net col0: track 323.8 -> 310.7 mm
- net Net-(D54-Pad2): track 48.9 -> 35.9 mm, vias 1 -> 0
- net Net-(D49-Pad2): track 57.7 -> 49.8 mm, vias 2 -> 0
- net LED: track 21.8 -> 14.5 mm
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Other:
- board text added: "PCB designed by ... t.komi"
- board text removed: "PCB designed by ... T.komiyama"
